Commit message: Fix urdf limit.

File: resources/robots/diablo/urdf/diablo_asm.urdf (robot description, URDF)
Before this commit: robot diablo_ASM, 7 links, 6 joints
Joints:
- joint left_fake_knee_joint: limit lower=-1.57 upper=1.57 effort=27 velocity=26 -> lower=0.0 upper=2.9 effort=27 velocity=26
- joint right_fake_knee_joint: limit lower=-1.57 upper=1.57 effort=27 velocity=26 -> lower=0.0 upper=2.9 effort=27 velocity=26

Commit message: Change wheel vel rewart to urdf vel limit.

File: resources/robots/diablo/urdf/diablo_asm.urdf (robot description, URDF)
Before this commit: robot diablo_ASM, 7 links, 6 joints
Joints:
- joint left_wheel_joint: limit effort=5 velocity=26 -> effort=5 velocity=5
- joint right_wheel_joint: limit effort=5 velocity=26 -> effort=5 velocity=5

Commit message: Use right urdf limit.

File: resources/robots/diablo/urdf/diablo_asm.urdf (robot description, URDF)
Before this commit: robot diablo_ASM, 7 links, 6 joints
Joints:
- joint left_wheel_joint: limit effort=5 velocity=5 -> effort=27 velocity=26
- joint right_wheel_joint: limit effort=5 velocity=5 -> effort=27 velocity=26

Commit message: Change low_limit.

File: resources/robots/diablo/urdf/diablo_asm.urdf (robot description, URDF)
Before this commit: robot diablo_ASM, 7 links, 6 joints
Joints:
- joint left_fake_knee_joint: limit lower=0.0 upper=2.9 effort=27 velocity=26 -> lower=-0.1 upper=2.9 effort=27 velocity=26
- joint right_fake_knee_joint: limit lower=0.0 upper=2.9 effort=27 velocity=26 -> lower=-0.1 upper=2.9 effort=27 velocity=26
